File: pcb/led-driver.sch (KiCad schematic (older format))
At the start: 14 parts, among them P201 CONN_01X02, P202 CONN_01X02, P203 CONN_01X02, Q201 AM4874N, Q202 AM4874N, Q203 AM4874N, U201 LM2902N, U202 MAX5813

Commit message: removed excess power pins. moved parts around.
Parts:
- removed C201, C205, C206: C, Capacitors_SMD:c_elec_3x5.3, symbol C
- added P204: CONN_01X01, netl:1Pin_big, symbol CONN_01X01
- added Q204: AM4874N, Housings_SOIC:SOIC-8_3.9x4.9mm_Pitch1.27mm, symbol AM4874N
- added R201: R, netl:SMD_0603, symbol R
- P201, P202, P203: value CONN_01X02 -> CONN_01X01; footprint Pin_Headers:Pin_Header_Straight_1x02 -> netl:1Pin_big; symbol CONN_01X02 -> CONN_01X01
Connections:
- net labels added: DrainWhite, W
- wire segments 55 -> 52
Other:
- moved on the sheet: R205, R206, U201B, U201C, U202

Commit message: added cap for opamp
Parts:
- added C201: C, netl:SMD_0603, symbol C
Connections:
- wire segments 52 -> 54
Changed lines of the file:
@@
 Connection ~ 3150 2050
 $Comp
-L GND #PWR014
+L GND #PWR013
 U 1 1 566DE548
 P 2200 2550
-F 0 "#PWR014" H 2200 2300 50  0001 C CNN
+F 0 "#PWR013" H 2200 2300 50  0001 C CNN
 F 1 "GND" H 2200 2400 50  0000 C CNN
 F 2 "" H 2200 2550 60  0000 C CNN
@@
 $EndComp
 $Comp
-L GND #PWR015
+L GND #PWR014
 U 1 1 566E450E
 P 3250 4850
-F 0 "#PWR015" H 3250 4600 50  0001 C CNN
+F 0 "#PWR014" H 3250 4600 50  0001 C CNN
 F 1 "GND" H 3250 4700 50  0000 C CNN
 F 2 "" H 3250 4850 60  0000 C CNN
@@
 Connection ~ 3150 4350
 $Comp
-L GND #PWR017
+L GND #PWR015
 U 1 1 566E453D
 P 2200 4850
-F 0 "#PWR017" H 2200 4600 50  0001 C CNN
+F 0 "#PWR015" H 2200 4600 50  0001 C CNN
 F 1 "GND" H 2200 4700 50  0000 C CNN
 F 2 "" H 2200 4850 60  0000 C CNN
@@
 $EndComp
 $Comp
-L GND #PWR018
+L GND #PWR016
 U 1 1 566E478C
 P 6400 2550
-F 0 "#PWR018" H 6400 2300 50  0001 C CNN
+F 0 "#PWR016" H 6400 2300 50  0001 C CNN
 F 1 "GND" H 6400 2400 50  0000 C CNN
 F 2 "" H 6400 2550 60  0000 C CNN
@@
 Connection ~ 6300 2050
 $Comp
-L GND #PWR020
+L GND #PWR017
 U 1 1 566E47BB
 P 5350 2550
-F 0 "#PWR020" H 5350 2300 50  0001 C CNN
+F 0 "#PWR017" H 5350 2300 50  0001 C CNN
 F 1 "GND" H 5350 2400 50  0000 C CNN
 F 2 "" H 5350 2550 60  0000 C CNN
@@
 B
 $Comp
-L GND #PWR021
+L GND #PWR018
 U 1 1 566E84F5
 P 3750 6450
-F 0 "#PWR021" H 3750 6200 50  0001 C CNN
+F 0 "#PWR018" H 3750 6200 50  0001 C CNN
 F 1 "GND" H 3750 6300 50  0000 C CNN
 F 2 "" H 3750 6450 60  0000 C CNN
@@
 	5000 6550 5150 6550
 $Comp
-L GND #PWR022
+L GND #PWR019
 U 1 1 566E8506
 P 5150 6750
-F 0 "#PWR022" H 5150 6500 50  0001 C CNN
+F 0 "#PWR019" H 5150 6500 50  0001 C CNN
 F 1 "GND" H 5150 6600 50  0000 C CNN
 F 2 "" H 5150 6750 60  0000 C CNN
@@
 $EndComp
 $Comp
-L GND #PWR023
+L GND #PWR020
 U 1 1 566E01A5
 P 6400 4850
-F 0 "#PWR023" H 6400 4600 50  0001 C CNN
+F 0 "#PWR020" H 6400 4600 50  0001 C CNN
 F 1 "GND" H 6400 4700 50  0000 C CNN
 F 2 "" H 6400 4850 60  0000 C CNN
@@
 Connection ~ 6300 4350
 $Comp
-L GND #PWR025
+L GND #PWR021
 U 1 1 566E01CE
 P 5350 4850
-F 0 "#PWR025" H 5350 4600 50  0001 C CNN
+F 0 "#PWR021" H 5350 4600 50  0001 C CNN
 F 1 "GND" H 5350 4700 50  0000 C CNN
 F 2 "" H 5350 4850 60  0000 C CNN
@@
 Wire Wire Line
 	4050 6650 3950 6650
+$Comp
+L C C201
+U 1 1 566EA826
+P 7750 2950
+F 0 "C201" H 7775 3050 50  0000 L CNN
+F 1 "C" H 7775 2850 50  0000 L CNN
+F 2 "netl:SMD_0603" H 7788 2800 30  0001 C CNN
+F 3 "" H 7750 2950 60  0000 C CNN
+	1    7750 2950
+	-1   0    0    1
+$EndComp
+Text GLabel 7750 2700 1    60   Input ~ 0
+Vdd
+$Comp
+L GND #PWR022
+U 1 1 566EAF9B
+P 7750 3200
+F 0 "#PWR022" H 7750 2950 50  0001 C CNN
+F 1 "GND" H 7750 3050 50  0000 C CNN
+F 2 "" H 7750 3200 60  0000 C CNN
+F 3 "" H 7750 3200 60  0000 C CNN
+	1    7750 3200
+	1    0    0    -1
+$EndComp
+Wire Wire Line
+	7750 3100 7750 3200
+Wire Wire Line
+	7750 2800 7750 2700
 $EndSCHEMATC

Commit message: changed fets, added usb serial
Parts:
- removed Q201, Q202, Q203, Q204: AM4874N, Housings_SOIC:SOIC-8_3.9x4.9mm_Pitch1.27mm, symbol AM4874N
- added Q201, Q202, Q203, Q204: Q_NMOS_GDSD, netl:TO252, symbol Q_NMOS_GDSD
- U201: footprint Housings_SSOP:SSOP-14_5.3x6.2mm_Pitch0.65mm -> Housings_SOIC:SOIC-14_3.9x8.7mm_Pitch1.27mm
- renumbered R204 to R201, R205 to R202, R206 to R203, R201 to R204
Other:
- moved on the sheet: P201, P202, P203, P204, R201, R202, R203, R204

Commit message: ready for etching!
Parts:
- added C202, C?: 100n, netl:SMD_0603, symbol C
- C201: value C -> 100n
Connections:
- net 3v3: now also C202.2, C?.2
- net GND: now also C202.1, C?.1
- net Vdd renamed 5V
Changed lines of the file:
@@
 $EndDescr
 $Comp
-L GND #PWR012
+L GND #PWR08
 U 1 1 566DBED0
 P 3200 2550
-F 0 "#PWR012" H 3200 2300 50  0001 C CNN
+F 0 "#PWR08" H 3200 2300 50  0001 C CNN
 F 1 "GND" H 3200 2400 50  0000 C CNN
 F 2 "" H 3200 2550 60  0000 C CNN
@@
 	1800 2050 1800 1800
 $Comp
-L GND #PWR013
+L GND #PWR09
 U 1 1 566DE548
 P 2200 2550
-F 0 "#PWR013" H 2200 2300 50  0001 C CNN
+F 0 "#PWR09" H 2200 2300 50  0001 C CNN
 F 1 "GND" H 2200 2400 50  0000 C CNN
 F 2 "" H 2200 2550 60  0000 C CNN
@@
 $EndComp
 Text GLabel 2200 1000 1    60   Input ~ 0
-Vdd
+5V
 Wire Wire Line
 	2200 1000 2200 1300
@@
 	3200 1250 3200 1500
 $Comp
-L GND #PWR014
+L GND #PWR010
 U 1 1 566E450E
 P 3200 4850
-F 0 "#PWR014" H 3200 4600 50  0001 C CNN
+F 0 "#PWR010" H 3200 4600 50  0001 C CNN
 F 1 "GND" H 3200 4700 50  0000 C CNN
 F 2 "" H 3200 4850 60  0000 C CNN
@@
 	1800 4350 1800 4100
 $Comp
-L GND #PWR015
+L GND #PWR011
 U 1 1 566E453D
 P 2200 4850
-F 0 "#PWR015" H 2200 4600 50  0001 C CNN
+F 0 "#PWR011" H 2200 4600 50  0001 C CNN
 F 1 "GND" H 2200 4700 50  0000 C CNN
 F 2 "" H 2200 4850 60  0000 C CNN
@@
 $EndComp
 Text GLabel 2200 3300 1    60   Input ~ 0
-Vdd
+5V
 Wire Wire Line
 	2200 3300 2200 3600
@@
 	3200 3550 3200 3800
 $Comp
-L GND #PWR016
+L GND #PWR012
 U 1 1 566E478C
 P 6350 2550
-F 0 "#PWR016" H 6350 2300 50  0001 C CNN
+F 0 "#PWR012" H 6350 2300 50  0001 C CNN
 F 1 "GND" H 6350 2400 50  0000 C CNN
 F 2 "" H 6350 2550 60  0000 C CNN
@@
 	4950 2050 4950 1800
 $Comp
-L GND #PWR017
+L GND #PWR013
 U 1 1 566E47BB
 P 5350 2550
-F 0 "#PWR017" H 5350 2300 50  0001 C CNN
+F 0 "#PWR013" H 5350 2300 50  0001 C CNN
 F 1 "GND" H 5350 2400 50  0000 C CNN
 F 2 "" H 5350 2550 60  0000 C CNN
@@
 $EndComp
 Text GLabel 5350 1000 1    60   Input ~ 0
-Vdd
+5V
 Wire Wire Line
 	5350 1000 5350 1300
@@
 $EndComp
 $Comp
-L GND #PWR018
+L GND #PWR014
 U 1 1 566E84F5
 P 3750 6450
-F 0 "#PWR018" H 3750 6200 50  0001 C CNN
+F 0 "#PWR014" H 3750 6200 50  0001 C CNN
 F 1 "GND" H 3750 6300 50  0000 C CNN
 F 2 "" H 3750 6450 60  0000 C CNN
@@
 Wire Wire Line
 	3950 6550 4050 6550
-Text GLabel 3950 6750 0    60   Input ~ 0
+Text GLabel 3800 6750 0    60   Input ~ 0
 3v3
 Wire Wire Line
-	3950 6750 4050 6750
-Text GLabel 5150 6150 2    60   Input ~ 0
+	3800 6750 4050 6750
+Text GLabel 5900 6150 2    60   Input ~ 0
 3v3
 Wire Wire Line
@@
 	5000 6550 5150 6550
 $Comp
-L GND #PWR019
+L GND #PWR015
 U 1 1 566E8506
 P 5150 6750
-F 0 "#PWR019" H 5150 6500 50  0001 C CNN
+F 0 "#PWR015" H 5150 6500 50  0001 C CNN
 F 1 "GND" H 5150 6600 50  0000 C CNN
 F 2 "" H 5150 6750 60  0000 C CNN
@@
 	5000 6750 5150 6750
 Wire Wire Line
-	5150 6150 5000 6150
+	5000 6150 5900 6150
 Wire Wire Line
 	5000 6150 5000 6350
@@
 DrainWhite
 $Comp
-L GND #PWR020
+L GND #PWR016
 U 1 1 566E01A5
 P 6350 4850
-F 0 "#PWR020" H 6350 4600 50  0001 C CNN
+F 0 "#PWR016" H 6350 4600 50  0001 C CNN
 F 1 "GND" H 6350 4700 50  0000 C CNN
 F 2 "" H 6350 4850 60  0000 C CNN
@@
 	4950 4350 4950 4100
 $Comp
-L GND #PWR021
+L GND #PWR017
 U 1 1 566E01CE
 P 5350 4850
-F 0 "#PWR021" H 5350 4600 50  0001 C CNN
+F 0 "#PWR017" H 5350 4600 50  0001 C CNN
 F 1 "GND" H 5350 4700 50  0000 C CNN
 F 2 "" H 5350 4850 60  0000 C CNN
@@
 $EndComp
 Text GLabel 5350 3300 1    60   Input ~ 0
-Vdd
+5V
 Wire Wire Line
 	5350 3300 5350 3600
@@
 P 7750 2950
 F 0 "C201" H 7775 3050 50  0000 L CNN
-F 1 "C" H 7775 2850 50  0000 L CNN
+F 1 "100n" H 7775 2850 50  0000 L CNN
 F 2 "netl:SMD_0603" H 7788 2800 30  0001 C CNN
 F 3 "" H 7750 2950 60  0000 C CNN
@@
 $EndComp
 Text GLabel 7750 2700 1    60   Input ~ 0
-Vdd
-$Comp
-L GND #PWR022
+5V
+$Comp
+L GND #PWR018
 U 1 1 566EAF9B
 P 7750 3200
-F 0 "#PWR022" H 7750 2950 50  0001 C CNN
+F 0 "#PWR018" H 7750 2950 50  0001 C CNN
 F 1 "GND" H 7750 3050 50  0000 C CNN
 F 2 "" H 7750 3200 60  0000 C CNN
@@
 Connection ~ 6350 1500
 Connection ~ 3200 1500
+$Comp
+L C C202
+U 1 1 56B91DE7
+P 5650 6300
+F 0 "C202" H 5675 6400 50  0000 L CNN
+F 1 "100n" H 5675 6200 50  0000 L CNN
+F 2 "netl:SMD_0603" H 5688 6150 30  0001 C CNN
+F 3 "" H 5650 6300 60  0000 C CNN
+	1    5650 6300
+	-1   0    0    1
+$EndComp
+$Comp
+L GND #PWR019
+U 1 1 56B92263
+P 5650 6550
+F 0 "#PWR019" H 5650 6300 50  0001 C CNN
+F 1 "GND" H 5650 6400 50  0000 C CNN
+F 2 "" H 5650 6550 60  0000 C CNN
+F 3 "" H 5650 6550 60  0000 C CNN
+	1    5650 6550
+	1    0    0    -1
+$EndComp
+Wire Wire Line
+	5650 6550 5650 6450
+Connection ~ 5650 6150
+$Comp
+L C C?
+U 1 1 56B92AE4
+P 3950 6900
+F 0 "C?" H 3975 7000 50  0000 L CNN
+F 1 "100n" H 3975 6800 50  0000 L CNN
+F 2 "netl:SMD_0603" H 3988 6750 30  0001 C CNN
+F 3 "" H 3950 6900 60  0000 C CNN
+	1    3950 6900
+	-1   0    0    1
+$EndComp
+Connection ~ 3950 6750
+$Comp
+L GND #PWR?
+U 1 1 56B92D0C
+P 3950 7100
+F 0 "#PWR?" H 3950 6850 50  0001 C CNN
+F 1 "GND" H 3950 6950 50  0000 C CNN
+F 2 "" H 3950 7100 60  0000 C CNN
+F 3 "" H 3950 7100 60  0000 C CNN
+	1    3950 7100
+	1    0    0    -1
+$EndComp
+Wire Wire Line
+	3950 7050 3950 7100
 $EndSCHEMATC
