File: pcb/mcu.sch (KiCad schematic (older format))
At the start: 0 parts

Commit message: added mcu
Parts:
- added C401: C, netl:SMD_0603, symbol C
- added IC401: ATMEGA48-M, Housings_QFP:TQFP-32_7x7mm_Pitch0.8mm, symbol ATMEGA48-M
- added P401, P402, P403, P404, P405, P406, P407, P408, P409, P410, P411, P412, P413, P414: CONN_01X01, netl:1Pin_small, symbol CONN_01X01
Connections:
- new net: IC401.1 ((PCINT19/OC2B/INT1)PD3), P410.1 (P1)
- new net: IC401.10 ((PCINT22/OC0A/AIN0)PD6), P413.1 (P1)
- new net: IC401.11 ((PCINT23/AIN1)PD7), P414.1 (P1)
- new net: IC401.12 ((PCINT0/CLKO/ICP1)PB0), P404.1 (P1)
- new net: IC401.13 ((PCINT1/OC1A)PB1), P405.1 (P1)
- new net: IC401.14 ((PCINT2/OC1B/~SS~)PB2), P406.1 (P1)
- new net: IC401.19 (ADC6), P402.1 (P1)
- new net: IC401.2 ((PCINT20/XCK/T0)PD4), P411.1 (P1)
- new net: IC401.20 (AREF), P401.1 (P1)
- new net: IC401.22 (ADC7), P403.1 (P1)
- new net: IC401.32 ((PCINT18/INT0)PD2), P409.1 (P1)
- new net: IC401.7 ((PCINT6/XTAL1/TOSC1)PB6), P407.1 (P1)
- new net: IC401.8 ((PCINT7/XTAL2/TOSC2)PB7), P408.1 (P1)
- new net: IC401.9 ((PCINT21/OC0B/T1)PD5), P412.1 (P1)
- new net 3v3: C401.1, IC401.18 (AVCC), IC401.4 (VCC), IC401.6 (VCC)
- new net GND: C401.2, IC401.21 (GND), IC401.3 (GND), IC401.5 (GND)
- new net MISO: IC401.16 ((PCINT4/MISO)PB4)
- new net MOSI: IC401.15 ((PCINT3/OC2/MOSI)PB3)
- new net PWMA: IC401.23 ((PCINT8/ADC0)PC0)
- new net PWMB: IC401.24 ((PCINT9/ADC1)PC1)
- new net PWMC: IC401.25 ((PCINT10/ADC2)PC2)
- new net PWMD: IC401.26 ((PCINT11/ADC3)PC3)
- new net RX: IC401.30 ((PCINT16/RXD)PD0)
- new net SCK: IC401.17 ((PCINT5/SCK)PB5)
- new net SCL: IC401.28 ((PCINT13/SCL/ADC5)PC5)
- new net SDA: IC401.27 ((PCINT12/SDA/ADC4)PC4)
- new net TX: IC401.31 ((PCINT17/TXD)PD1)
- new net ~RESET: IC401.29 ((PCINT14/~RESET~)PC6)
