File: pcb/rpi_shield.kicad_pcb (KiCad board)
At the start: 2 copper layers, 65 x 56 mm, 113 parts, among them IC401 ATMEGA48-M, P101 CONN_01X08, P102 CONN_02X20, P301 USB_OTG, P401 CONN_01X01, P402 CONN_01X01, P403 CONN_01X01, P404 CONN_01X01, P405 CONN_01X01, P406 CONN_01X01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

Commit message: working version from assembly 2016
Parts:
- removed the VIA at (157.7, 107.6)
- removed the VIA at (157.7, 102.4)
- removed the VIA at (140.9, 103.2)
- removed the VIA at (177.1, 108.6)
- moved G*** 18.5 mm to (194.4, 100.6) (x2)
- moved P101 6.83 mm to (147.0, 136.0)
Routing:
- net Net-(R215-Pad2): track 44.0 -> 45.4 mm
- net Net-(Q201-Pad3): track 58.4 -> 59.1 mm
- net /LED driver/PWMA: track 39.8 -> 39.1 mm
- net Net-(Q204-Pad3): track 29.9 -> 29.4 mm
Other:
- net class Default: clearance 0.2 -> 0.4
- rule trace_clearance: 0.2 -> 0.4
